Commit message: Update Gazebo top view and arm visuals

File: src/my_robot_description/urdf/arm.xacro (robot description, xacro)
@@ -1,77 +1,80 @@
 <?xml version="1.0"?>
 <robot xmlns:xacro="http://www.ros.org/wiki/xacro">
-    <xacro:property name="arm_base_length" value="0.1" />
-    <xacro:property name="arm_base_width" value="0.1" />
-    <xacro:property name="arm_base_height" value="0.02" />
-    <xacro:property name="forearm_radius" value="0.02" />
-    <xacro:property name="forearm_length" value="0.3" />
-    <xacro:property name="hand_link_radius" value="0.02" />
-    <xacro:property name="hand_link_length" value="0.3" />
-    <link name="arm_base_link">
+    <xacro:property name="omx_base_radius" value="0.045" />
+    <xacro:property name="omx_base_height" value="0.040" />
+    <xacro:property name="omx_shoulder_radius" value="0.030" />
+    <xacro:property name="omx_shoulder_height" value="0.0595" />
+    <xacro:property name="omx_upper_arm_length" value="0.128" />
+    <xacro:property name="omx_upper_arm_radius" value="0.020" />
+    <xacro:property name="omx_forearm_length" value="0.124" />
+    <xacro:property name="omx_forearm_radius" value="0.018" />
+    <xacro:property name="omx_wrist_length" value="0.082" />
+    <xacro:property name="omx_wrist_width" value="0.045" />
+    <xacro:property name="omx_wrist_height" value="0.040" />
+    <xacro:property name="omx_finger_length" value="0.060" />
+    <xacro:property name="omx_finger_width" value="0.010" />
+    <xacro:property name="omx_finger_height" value="0.018" />
+    <xacro:property name="omx_finger_gap" value="0.042" />
+    <xacro:property name="omx_upper_arm_pitch" value="${pi / 3.0}" />
+    <xacro:property name="omx_forearm_pitch" value="${pi / 3.6}" />
+    <xacro:macro name="open_manipulator_visual_arm" params="mount_x mount_y mount_z">
+        <xacro:property name="arm_stack_top_z" value="${mount_z + omx_base_height + omx_shoulder_height}" />
+        <xacro:property name="upper_half_x" value="${omx_upper_arm_length * sin(omx_upper_arm_pitch) / 2.0}" />
+        <xacro:property name="upper_half_z" value="${omx_upper_arm_length * cos(omx_upper_arm_pitch) / 2.0}" />
+        <xacro:property name="upper_tip_x" value="${mount_x + omx_upper_arm_length * sin(omx_upper_arm_pitch)}" />
+        <xacro:property name="upper_tip_z" value="${arm_stack_top_z + omx_upper_arm_length * cos(omx_upper_arm_pitch)}" />
+        <xacro:property name="forearm_half_x" value="${omx_forearm_length * sin(omx_forearm_pitch) / 2.0}" />
+        <xacro:property name="forearm_half_z" value="${omx_forearm_length * cos(omx_forearm_pitch) / 2.0}" />
+        <xacro:property name="forearm_tip_x" value="${upper_tip_x + omx_forearm_length * sin(omx_forearm_pitch)}" />
+        <xacro:property name="forearm_tip_z" value="${upper_tip_z + omx_forearm_length * cos(omx_forearm_pitch)}" />
         <visual>
             <geometry>
-                <box size="${arm_base_length} ${arm_base_width} ${arm_base_height}" />
+                <cylinder radius="${omx_base_radius}" length="${omx_base_height}" />
             </geometry>
-            <origin xyz="0 0 ${arm_base_height / 2}" rpy="0 0 0" />
-            <material name="orange" />
+            <origin xyz="${mount_x} ${mount_y} ${mount_z + omx_base_height / 2.0}" rpy="0 0 0" />
+            <material name="arm_graphite" />
         </visual>
-        <collision>
-            <geometry>
-                <box size="${arm_base_length} ${arm_base_width} ${arm_base_height}" />
-            </geometry>
-            <origin xyz="0 0 ${arm_base_height / 2}" rpy="0 0 0" />
-        </collision>
-        <xacro:box_inertia m="0.5" l="${2*arm_base_length}" w="${2*arm_base_width}" h="${2*arm_base_height}"
-                            xyz="0 0 ${arm_base_height / 2}" rpy="0 0 0" />
-    </link>
-    <link name="forearm_link">
         <visual>
             <geometry>
-                <cylinder radius="${forearm_radius}" length="${forearm_length}" />
+                <cylinder radius="${omx_shoulder_radius}" length="${omx_shoulder_height}" />
             </geometry>
-            <origin xyz="0 0 ${forearm_length/2}" rpy="0 0 0" />
-            <material name="yellow" />
+            <origin xyz="${mount_x} ${mount_y} ${mount_z + omx_base_height + omx_shoulder_height / 2.0}" rpy="0 0 0" />
+            <material name="arm_copper" />
         </visual>
-        <collision>
-            <geometry>
-                <cylinder radius="${forearm_radius}" length="${forearm_length}" />
-            </geometry>
-            <origin xyz="0 0 ${forearm_length/2}" rpy="0 0 0" />
-        </collision>
-        <xacro:cylinder_inertia m="0.3" r="${2*forearm_radius}" h="${2*forearm_length}"
-                                xyz="0 0 ${forearm_length/2}" rpy="0 0 0" />
-    </link>
-    <link name="hand_link">
         <visual>
             <geometry>
-                <cylinder radius="${hand_link_radius}" length="${hand_link_length}" />
+                <cylinder radius="${omx_upper_arm_radius}" length="${omx_upper_arm_length}" />
             </geometry>
-            <origin xyz="0 0 ${hand_link_length / 2}" rpy="0 0 0" />
-            <material name="orange" />
+            <origin xyz="${mount_x + upper_half_x} ${mount_y} ${arm_stack_top_z + upper_half_z}" rpy="0 ${omx_upper_arm_pitch} 0" />
+            <material name="arm_sand" />
         </visual>
-        <collision>
+        <visual>
             <geometry>
-                <cylinder radius="${hand_link_radius}" length="${hand_link_length}" />
+                <cylinder radius="${omx_forearm_radius}" length="${omx_forearm_length}" />
             </geometry>
-            <origin xyz="0 0 ${hand_link_length / 2}" rpy="0 0 0" />
-        </collision>
-        <xacro:cylinder_inertia m="0.3" r="${2*forearm_radius}" h="${2*forearm_length}"
-                                xyz="0 0 ${forearm_length/2}" rpy="0 0 0" />
-    </link>
-    <joint name="arm_base_forearm_joint" type="revolute">
-        <parent link="arm_base_link" />
-        <child link="forearm_link" />
-        <origin xyz="0 0 ${arm_base_height}" rpy="0 0 0" />
-        <axis xyz="0 1 0" />
-        <limit lower="0" upper="${pi/2}" effort="100" velocity="100" />
-        <dynamics friction="0.5" damping="0.1" />
-    </joint>
-    <joint name="forearm_hand_joint" type="revolute">
-        <parent link="forearm_link" />
-        <child link="hand_link" />
-        <origin xyz="0 0 ${hand_link_length}" rpy="0 0 0" />
-        <axis xyz="0 1 0" />
-        <limit lower="0" upper="${pi/2}" effort="100" velocity="100" />
-        <dynamics friction="0.5" damping="0.1" />
-    </joint>
+            <origin xyz="${upper_tip_x + forearm_half_x} ${mount_y} ${upper_tip_z + forearm_half_z}" rpy="0 ${omx_forearm_pitch} 0" />
+            <material name="arm_graphite" />
+        </visual>
+        <visual>
+            <geometry>
+                <box size="${omx_wrist_length} ${omx_wrist_width} ${omx_wrist_height}" />
+            </geometry>
+            <origin xyz="${forearm_tip_x + omx_wrist_length / 2.0} ${mount_y} ${forearm_tip_z}" rpy="0 0 0" />
+            <material name="arm_copper" />
+        </visual>
+        <visual>
+            <geometry>
+                <box size="${omx_finger_length} ${omx_finger_width} ${omx_finger_height}" />
+            </geometry>
+            <origin xyz="${forearm_tip_x + omx_wrist_length + omx_finger_length / 2.0} ${mount_y + omx_finger_gap / 2.0} ${forearm_tip_z}" rpy="0 0 0" />
+            <material name="arm_graphite" />
+        </visual>
+        <visual>
+            <geometry>
+                <box size="${omx_finger_length} ${omx_finger_width} ${omx_finger_height}" />
+            </geometry>
+            <origin xyz="${forearm_tip_x + omx_wrist_length + omx_finger_length / 2.0} ${mount_y - omx_finger_gap / 2.0} ${forearm_tip_z}" rpy="0 0 0" />
+            <material name="arm_graphite" />
+        </visual>
+    </xacro:macro>
 </robot>

File: src/my_robot_description/urdf/common_properties.xacro (robot description, xacro)
@@ -15,4 +15,13 @@
     <material name="yellow">
         <color rgba="1.0 1.0 0 1" />
+    </material>
+    <material name="arm_copper">
+        <color rgba="0.82 0.38 0.10 1" />
+    </material>
+    <material name="arm_sand">
+        <color rgba="0.92 0.78 0.22 1" />
+    </material>
+    <material name="arm_graphite">
+        <color rgba="0.25 0.27 0.30 1" />
     </material>
     <xacro:macro name="box_inertia" params="m l w h xyz rpy" >

File: src/my_robot_description/urdf/mobile_base_gazebo.xacro (robot description, xacro)
@@ -1,7 +1,4 @@
 <?xml version="1.0"?>
 <robot xmlns:xacro="http://www.ros.org/wiki/xacro">
-    <gazebo reference="base_link">
-        <material>Gazebo/Blue</material>
-    </gazebo>
     <gazebo reference="right_wheel_link">
         <material>Gazebo/Red</material>
@@ -25,4 +22,7 @@
             <wheel_separation>0.45</wheel_separation>
             <wheel_diameter>0.2</wheel_diameter>
+            <!-- limits -->
+            <max_wheel_torque>8.0</max_wheel_torque>
+            <max_wheel_acceleration>0.6</max_wheel_acceleration>
             <!-- output -->
             <publish_odom>true</publish_odom>
@@ -31,5 +31,5 @@
             <odometry_topic>odom</odometry_topic>
             <odometry_frame>odom</odometry_frame>
-            <robot_base_frame>chassis</robot_base_frame>
+            <robot_base_frame>base_footprint</robot_base_frame>
         </plugin>
     </gazebo>
